Commit message: first commit

File: turtlebot3_description/urdf/turtlebot3_burger.urdf.xacro (robot description, xacro)
@@ -1,142 +1,327 @@
 <?xml version="1.0" ?>
-<robot name="turtlebot3_burger" xmlns:xacro="http://ros.org/wiki/xacro">
-  <xacro:include filename="$(find turtlebot3_description)/urdf/common_properties.xacro"/>
-  <xacro:include filename="$(find turtlebot3_description)/urdf/turtlebot3_burger.gazebo.xacro"/>
-  <link name="base_footprint"/>
-  <joint name="base_joint" type="fixed">
-    <parent link="base_footprint"/>
-    <child link="base_link"/>
-    <origin xyz="0.0 0.0 0.010" rpy="0 0 0"/>
-  </joint>
-  <link name="base_link">
-    <visual>
-      <origin xyz="-0.032 0 0.0" rpy="0 0 0"/>
-      <geometry>
-        <mesh filename="package://turtlebot3_description/meshes/bases/burger_base.stl" scale="0.001 0.001 0.001"/>
-      </geometry>
-      <material name="light_black"/>
-    </visual>
-    <collision>
-      <origin xyz="-0.032 0 0.070" rpy="0 0 0"/>
-      <geometry>
-        <box size="0.140 0.140 0.143"/>
-      </geometry>
-    </collision>
-    <inertial>
-      <origin xyz="0 0 0" rpy="0 0 0"/>
-      <mass value="8.2573504e-01"/>
-      <inertia ixx="2.2124416e-03" ixy="-1.2294101e-05" ixz="3.4938785e-05"
-               iyy="2.1193702e-03" iyz="-5.0120904e-06"
-               izz="2.0064271e-03" />
-    </inertial>
-  </link>
-  <joint name="wheel_left_joint" type="continuous">
-    <parent link="base_link"/>
-    <child link="wheel_left_link"/>
-    <origin xyz="0.0 0.08 0.023" rpy="-1.57 0 0"/>
-    <axis xyz="0 0 1"/>
-  </joint>
-  <link name="wheel_left_link">
-    <visual>
-      <origin xyz="0 0 0" rpy="1.57 0 0"/>
-      <geometry>
-        <mesh filename="package://turtlebot3_description/meshes/wheels/left_tire.stl" scale="0.001 0.001 0.001"/>
-      </geometry>
-      <material name="dark"/>
-    </visual>
-    <collision>
-      <origin xyz="0 0 0" rpy="0 0 0"/>
-      <geometry>
-        <cylinder length="0.018" radius="0.033"/>
-      </geometry>
-    </collision>
-    <inertial>
-      <origin xyz="0 0 0" />
-      <mass value="2.8498940e-02" />
-      <inertia ixx="1.1175580e-05" ixy="-4.2369783e-11" ixz="-5.9381719e-09"
-               iyy="1.1192413e-05" iyz="-1.4400107e-11"
-               izz="2.0712558e-05" />
-      </inertial>
-  </link>
-  <joint name="wheel_right_joint" type="continuous">
-    <parent link="base_link"/>
-    <child link="wheel_right_link"/>
-    <origin xyz="0.0 -0.080 0.023" rpy="-1.57 0 0"/>
-    <axis xyz="0 0 1"/>
-  </joint>
-  <link name="wheel_right_link">
-    <visual>
-      <origin xyz="0 0 0" rpy="1.57 0 0"/>
-      <geometry>
-        <mesh filename="package://turtlebot3_description/meshes/wheels/right_tire.stl" scale="0.001 0.001 0.001"/>
-      </geometry>
-      <material name="dark"/>
-    </visual>
-    <collision>
-      <origin xyz="0 0 0" rpy="0 0 0"/>
-      <geometry>
-        <cylinder length="0.018" radius="0.033"/>
-      </geometry>
-    </collision>
-    <inertial>
-      <origin xyz="0 0 0" />
-      <mass value="2.8498940e-02" />
-      <inertia ixx="1.1175580e-05" ixy="-4.2369783e-11" ixz="-5.9381719e-09"
-               iyy="1.1192413e-05" iyz="-1.4400107e-11"
-               izz="2.0712558e-05" />
-      </inertial>
-  </link>
-  <joint name="caster_back_joint" type="fixed">
-    <parent link="base_link"/>
-    <child link="caster_back_link"/>
-    <origin xyz="-0.081 0 -0.004" rpy="-1.57 0 0"/>
-  </joint>
-  <link name="caster_back_link">
-    <collision>
-      <origin xyz="0 0.001 0" rpy="0 0 0"/>
-      <geometry>
-        <box size="0.030 0.009 0.020"/>
-      </geometry>
-    </collision>
-    <inertial>
-      <origin xyz="0 0 0" />
-      <mass value="0.005" />
-      <inertia ixx="0.001" ixy="0.0" ixz="0.0"
-               iyy="0.001" iyz="0.0"
-               izz="0.001" />
-    </inertial>
-  </link>
-  <joint name="imu_joint" type="fixed">
-    <parent link="base_link"/>
-    <child link="imu_link"/>
-    <origin xyz="-0.032 0 0.068" rpy="0 0 0"/>
-  </joint>
-  <link name="imu_link"/>
-  <joint name="scan_joint" type="fixed">
-    <parent link="base_link"/>
-    <child link="base_scan"/>
-    <origin xyz="-0.032 0 0.172" rpy="0 0 0"/>
-  </joint>
-  <link name="base_scan">
-    <visual>
-      <origin xyz="0 0 0.0" rpy="0 0 0"/>
-      <geometry>
-        <mesh filename="package://turtlebot3_description/meshes/sensors/lds.stl" scale="0.001 0.001 0.001"/>
-      </geometry>
-      <material name="dark"/>
-    </visual>
-    <collision>
-      <origin xyz="0.015 0 -0.0065" rpy="0 0 0"/>
-      <geometry>
-        <cylinder length="0.0315" radius="0.055"/>
-      </geometry>
-    </collision>
-    <inertial>
-      <mass value="0.114" />
-      <origin xyz="0 0 0" />
-      <inertia ixx="0.001" ixy="0.0" ixz="0.0"
-               iyy="0.001" iyz="0.0"
-               izz="0.001" />
-    </inertial>
-  </link>
+<robot name="test_robot" xmlns:xacro="http://ros.org/wiki/xacro">
+    <material name="black">
+        <color rgba="0.0 0.0 0.0 0.7"/>
+    </material>
+    <material name="orange">
+        <color rgba="0.8 0.5 0.03 1.0"/>
+    </material>
+    <material name="sliver">
+        <color rgba="1.0 1.0 1.0 0.4"/>
+    </material>
+    <material name="sliver_1">
+        <color rgba="0.9 0.8 0.7 1.0"/>
+    </material>
+    <material name="red">
+        <color rgba="1 0.0 0.0 1.0"/>
+    </material>
+    <link name="base_footprint"/>
+    <joint name="base_joint" type="fixed">
+        <parent link="base_footprint"/>
+        <child link="base_link"/>
+        <origin xyz="0.0 0.0 0.0395" rpy="0 0 0"/>
+    </joint>
+    <link name="base_link">
+        <visual>
+        <origin xyz="0.0 0.0 0.0" rpy="0 0 0"/>
+        <geometry>
+        <box size="0.3970 0.319 0.003"/>
+        </geometry>
+        <material name="black"/>
+        </visual>
+        <collision>
+        <origin xyz="0.0 0.0 0.0" rpy="0 0 0"/>
+        <geometry>
+        <box size="0.3970 0.3970 0.003"/>
+        </geometry>
+        </collision>
+    </link>
+    <joint name="header_joint" type="fixed">
+        <parent link="base_link"/>
+        <child link="header_link"/>
+        <origin xyz="0.0 0.0 0.151" rpy="0 0 0"/>
+    </joint>
+    <link name="header_link">
+        <visual>
+        <origin xyz="0.0 0.0 0.0" rpy="0 0 0"/>
+        <geometry>
+        <box size="0.3970 0.319 0.003"/>
+        </geometry>
+        <material name="black"/>
+        </visual>
+        <collision>
+        <origin xyz="0.0 0.0 0.0" rpy="0 0 0"/>
+        <geometry>
+        <box size="0.3970 0.319 0.003"/>
+        </geometry>
+        </collision>
+    </link>
+    <joint name="imu_joint" type="fixed">
+        <parent link="header_link"/>
+        <child link="imu_link"/>
+        <origin xyz="0.0 0.0 0.005" rpy="0 0 0"/>
+    </joint>
+    <link name="imu_link">
+        <visual>
+        <origin xyz="0.0 0.0 0.0" rpy="0 0 0"/>
+        <geometry>
+        <box size="0.03 0.02 0.01"/>
+        </geometry>
+        <material name="red"/>
+        </visual>
+        <collision>
+        <origin xyz="0.0 0.0 0.0" rpy="0 0 0"/>
+        <geometry>
+        <box size="0.03 0.02 0.01"/>
+        </geometry>
+        </collision>
+    </link>
+    <joint name="wheel_left_joint" type="continuous">
+        <parent link="base_link"/>
+        <child link="wheel_left_link"/>
+        <origin xyz="0.0 -0.1505 0.023" rpy="1.57 0.0 0.0"/>
+        <axis xyz="0 0 1"/>
+    </joint>
+    <link name="wheel_left_link">
+        <visual>
+        <origin xyz="0.0 0.0 0.0" rpy="0.0 0.0 0.0"/>
+        <geometry>
+        <cylinder length="0.018" radius="0.0625"/>
+        </geometry>
+        <material name="orange"/>
+        </visual>
+        <collision>
+        <origin xyz="0.0 0.0 0.0" rpy="0.0 0.0 0.0"/>
+        <geometry>
+            <cylinder length="0.018" radius="0.0625"/>
+        </geometry>
+        </collision>
+    </link>
+    <joint name="wheel_right_joint" type="continuous">
+        <parent link="base_link"/>
+        <child link="wheel_right_link"/>
+        <origin xyz="0.0 0.15052 0.023" rpy="1.57 0.0 0.0"/>
+        <axis xyz="0 0 1"/>
+    </joint>
+    <link name="wheel_right_link">
+        <visual>
+        <origin xyz="0.0 0.0 0.0" rpy="0.0 0.0 0.0"/>
+        <geometry>
+        <cylinder length="0.018" radius="0.0625"/>
+        </geometry>
+        <material name="orange"/>
+        </visual>
+        <collision>
+        <origin xyz="0.0 0.0 0.0" rpy="0.0 0.0 0.0"/>
+        <geometry>
+            <cylinder length="0.018" radius="0.0625"/>
+        </geometry>
+        </collision>
+    </link>
+    <link name="base_scan">
+        <visual>
+        <origin xyz="0.0 0.0 0.01" rpy="0.0 0.0 0.0"/>
+        <geometry>
+        <cylinder length="0.02" radius="0.0315"/>
+        </geometry>
+        <material name="sliver_1"/>
+        </visual>
+        <collision>
+        <origin xyz="0.0 0.0 0.01" rpy="0.0 0.0 0.0"/>
+        <geometry>
+        <cylinder length="0.02" radius="0.0315"/>
+        </geometry>
+        </collision>
+    </link>
+    <joint name="ridar_joint" type="fixed">
+        <parent link="ridar_base_link"/>
+        <child link="base_scan"/>
+        <origin xyz="0.0 0.0 0.0 " rpy="0.0 0.0 0.0"/>
+        <axis xyz="0 0 1"/>
+    </joint>
+    <link name="suport_link_1">
+        <visual>
+        <origin xyz="0.0 0.0 0.0755" rpy="0.0 0.0 0.0"/>
+        <geometry>
+        <cylinder length="0.151" radius="0.005"/>
+        </geometry>
+        <material name="sliver"/>
+        </visual>
+        <collision>
+        <origin xyz="0.0 0.0 0.0755" rpy="0.0 0.0 0.0"/>
+        <geometry>
+        <cylinder length="0.151" radius="0.005"/>
+        </geometry>
+        </collision>
+    </link>
+    <joint name="suport_joint_1" type="fixed">
+        <parent link="base_link"/>
+        <child link="suport_link_1"/>
+        <origin xyz="-0.19 -0.15 0.0 " rpy="0.0 0.0 0.0"/>
+    </joint>
+    <link name="suport_link_2">
+        <visual>
+        <origin xyz="0.0 0.0 0.0755" rpy="0.0 0.0 0.0"/>
+        <geometry>
+        <cylinder length="0.151" radius="0.005"/>
+        </geometry>
+        <material name="sliver"/>
+        </visual>
+        <collision>
+        <origin xyz="0.0 0.0 0.0755" rpy="0.0 0.0 0.0"/>
+        <geometry>
+        <cylinder length="0.151" radius="0.005"/>
+        </geometry>
+        </collision>
+    </link>
+    <joint name="suport_joint_2" type="fixed">
+        <parent link="base_link"/>
+        <child link="suport_link_2"/>
+        <origin xyz="0.19 -0.15 0.0 " rpy="0.0 0.0 0.0"/>
+    </joint>
+    <link name="suport_link_3">
+        <visual>
+        <origin xyz="0.0 0.0 0.0755" rpy="0.0 0.0 0.0"/>
+        <geometry>
+        <cylinder length="0.151" radius="0.005"/>
+        </geometry>
+        <material name="sliver"/>
+        </visual>
+        <collision>
+        <origin xyz="0.0 0.0 0.0755" rpy="0.0 0.0 0.0"/>
+        <geometry>
+        <cylinder length="0.151" radius="0.005"/>
+        </geometry>
+        </collision>
+    </link>
+    <joint name="suport_joint_3" type="fixed">
+        <parent link="base_link"/>
+        <child link="suport_link_3"/>
+        <origin xyz="-0.19 0.15 0.0 " rpy="0.0 0.0 0.0"/>
+    </joint>
+    <link name="suport_link_4">
+        <visual>
+        <origin xyz="0.0 0.0 0.0755" rpy="0.0 0.0 0.0"/>
+        <geometry>
+        <cylinder length="0.151" radius="0.005"/>
+        </geometry>
+        <material name="sliver"/>
+        </visual>
+        <collision>
+        <origin xyz="0.0 0.0 0.0755" rpy="0.0 0.0 0.0"/>
+        <geometry>
+        <cylinder length="0.151" radius="0.005"/>
+        </geometry>
+        </collision>
+    </link>
+    <joint name="suport_joint_4" type="fixed">
+        <parent link="base_link"/>
+        <child link="suport_link_4"/>
+        <origin xyz="0.19 0.15 0.0 " rpy="0.0 0.0 0.0"/>
+    </joint>
+    <link name="ridar_base_link">
+        <visual>
+        <origin xyz="0.0 0.0 0.0" rpy="0.0 0.0 0.0"/>
+        <geometry>
+        <box size="0.12 0.08 0.003"/>
+        </geometry>
+        <material name="black"/>
+        </visual>
+        <collision>
+        <origin xyz="0.0 0.0 0.0" rpy="0.0 0.0 0.0"/>
+        <geometry>
+        <box size="0.3970 0.3970 0.003"/>
+        </geometry>
+        </collision>
+    </link>
+    <joint name="ridar_base_joint" type="fixed">
+        <parent link="header_link"/>
+        <child link="ridar_base_link"/>
+        <origin xyz="0.0 0.0 0.03 " rpy="0.0 0.0 0.0"/>
+        <axis xyz="0 0 1"/>
+    </joint>
+    <link name="suport_link_10">
+        <visual>
+        <origin xyz="0.0 0.0 0.015" rpy="0.0 0.0 0.0"/>
+        <geometry>
+        <cylinder length="0.03" radius="0.003"/>
+        </geometry>
+        <material name="sliver"/>
+        </visual>
+        <collision>
+        <origin xyz="0.0 0.0 0.0755" rpy="0.0 0.0 0.0"/>
+        <geometry>
+        <cylinder length="0.151" radius="0.005"/>
+        </geometry>
+        </collision>
+    </link>
+    <joint name="suport_joint_10" type="fixed">
+        <parent link="header_link"/>
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